File: Schematics/Coil_Circuitry/Coil_Circuitry.kicad_sch (KiCad schematic)
At the start: 1 part, among them Q1 Q_NMOS_DGS

Commit message: first draft circuit
Parts:
- removed Q1: Q_NMOS_DGS, symbol Device:Q_NMOS_DGS
- added D2: 1N914WT, Diode_SMD:D_SOD-523, symbol Diode:1N914WT
- added D3: LED, symbol Device:LED
- added J1: Conn_01x04_Pin, symbol Connector:Conn_01x04_Pin
- added L2: Coil, symbol Device:L
- added Q1: PMOS, symbol Simulation_SPICE:PMOS
- added Q2: NMOS, symbol Simulation_SPICE:NMOS
- added R1, R3: 4.7k, symbol Device:R_Small
- added R2, R6: 10k, symbol Device:R_Small
- added R4: 4,7k, symbol Device:R_Small
- added R5: R_Photo, symbol Device:R_Photo
- added R7: R_Variable, symbol Device:R_Variable
- added SW2: Manual, symbol Switch:SW_Push
Connections:
- new net: Q1.3 (S), R2.2
- new net: D3.2 (A), R4.2
- new net: R3.1, SW2.1
- new net: D2.2 (A), L2.2, Q2.1 (D)
- new net Act_Coil: Q1.1 (D), Q2.2 (G), R5.1, R6.2, R7.2, SW2.2
- new net Controlled_Coil: J1.4 (Pin_4), Q1.2 (G), R1.1
- new net GND: D3.1 (K), J1.2 (Pin_2), Q2.3 (S), R1.2, R5.2, R7.1
- new net Pres_Sensor: J1.3 (Pin_3)
- new net VCC: D2.1 (K), J1.1 (Pin_1), L2.1, R2.1, R3.2, R4.1, R6.1
Other:
- note added: "VDD"

Commit message: test
Parts:
- added U1: MOUDLE-SEEEDUINO-XIAO-ESP32C3, MOUDLE14P-SMD-2.54-21X17.8MM, symbol MOUDLE-SEEEDUINO-XIAO-ESP32C3:MOUDLE-SEEEDUINO-XIAO-ESP32C3
Changed lines of the file:
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@@
+    )
+  )
+  (symbol (lib_id "MOUDLE-SEEEDUINO-XIAO-ESP32C3:MOUDLE-SEEEDUINO-XIAO-ESP32C3") (at 49.53 105.41 0) (unit 1)
+    (in_bom yes) (on_board yes) (dnp no) (fields_autoplaced)
+    (property "Reference" "U1" (at 48.895 86.36 0)
+      (effects (font (size 1.27 1.27)))
+    )
+    (property "Value" "MOUDLE-SEEEDUINO-XIAO-ESP32C3" (at 48.895 88.9 0)
+      (effects (font (size 1.27 1.27)))
+    )
+    (property "Footprint" "MOUDLE14P-SMD-2.54-21X17.8MM" (at 49.53 105.41 0)
+      (effects (font (size 1.27 1.27)) (justify bottom) hide)
+    )
+    (property "Datasheet" "" (at 49.53 105.41 0)
+      (effects (font (size 1.27 1.27)) hide)
+    )
+    (pin "9")
+    (pin "8")
+    (pin "6")
+    (pin "3")
+    (pin "11")
+    (pin "10")
+    (pin "12")
+    (pin "13")
+    (pin "14")
+    (pin "2")
+    (pin "1")
+    (pin "5")
+    (pin "7")
+    (pin "4")
+    (instances
+      (project "Coil_Circuitry"
+        (path "/f0d7dc79-2865-4dd1-b2c5-de9bb2b6a418"
+          (reference "U1") (unit 1)
+        )
+      )
     )
   )

Commit message: fegcv
Parts:
- removed R7: R_Variable, symbol Device:R_Variable
- removed U1: MOUDLE-SEEEDUINO-XIAO-ESP32C3, MOUDLE14P-SMD-2.54-21X17.8MM, symbol MOUDLE-SEEEDUINO-XIAO-ESP32C3:MOUDLE-SEEEDUINO-XIAO-ESP32C3
- added JP1: Jumper_2_Open, symbol Jumper:Jumper_2_Open
- added JP2: Jumper_2_Open, Connector_PinHeader_1.00mm:PinHeader_1x02_P1.00mm_Vertical, symbol Jumper:Jumper_2_Open
- added R8: R_Variable, symbol Device:R_Variable
- J1: footprint (none) -> Connector_JST:JST_XH_B4B-XH-A_1x04_P2.50mm_Vertical; Note (none) -> JST Connector
Connections:
- net Act_Coil: now also JP1.2 (B), JP2.1 (A); no longer Q1.1 (D), R5.1, R6.2
- net Pres_Sensor: now also R5.1, R6.2, JP1.1 (A), R8.1
- net VCC: now also R2.2, R8.2; no longer R2.1
- net at Q1.3 (S): now also R2.1; no longer R2.2
- new net: JP2.2 (B), Q1.1 (D)
Other:
- moved on the sheet: D2, D3, L2, Q1, Q2, R1, R2, R3, R4, R5, R6, SW2

Commit message: photodiode
Parts:
- removed R5: R_Photo, symbol Device:R_Photo
- removed R6: 10k, symbol Device:R_Small
- removed R8: R_Variable, symbol Device:R_Variable
- added D1: D_Photo, symbol Device:D_Photo
- added R5: Optional, symbol Device:R_Small
- added R7: R_Variable, symbol Device:R_Variable
- D3: value LED -> IR LED
Connections:
- net GND: now also R5.2, R7.1
- net Pres_Sensor: now also D1.2 (A), R5.1, R7.2
- net VCC: now also D1.1 (K)
