File: Schematics/Elproj2V1/Elproj2V1.kicad_sch (KiCad schematic)
At the start: 83 parts, among them J1 Conn_01x04_Pin, J10 5V Barrel, J11 Conn_01x10_Pin, J12 CONN BUCK ON MAIN, J13 BUCK STAB CONN ON CARD, J14 BUCK CARD STAB CONN ON MAIN, J2 Conn_01x04_Pin, J3 Conn_01x04_Pin, J4 Conn_01x04_Pin, J5 Conn_01x04_Pin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

Commit message: Updated labels, references and mistakes
Parts:
- added R22, R23, R24: 10, symbol Device:R_Small
Connections:
- net Cap_PWR: now also J11.1 (Pin_1)
- net GNDPWR: now also J11.4 (Pin_4), J11.5 (Pin_5), U1.13 (GND); no longer J11.9 (Pin_9), J2.2 (Pin_2), J3.2 (Pin_2), J4.2 (Pin_2), J5.2 (Pin_2)
- net MAIN_FB: now also J11.2 (Pin_2)
- net MAIN_VOUT: now also J11.3 (Pin_3), J2.1 (Pin_1), J3.1 (Pin_1), J4.1 (Pin_1), J5.1 (Pin_1)
- net at U1.8 (PB09_A7_D7_RX): now also R22.2
- removed net Cap_BOOSTED_PWR: J11.8 (Pin_8), J2.1 (Pin_1), J3.1 (Pin_1), J4.1 (Pin_1), J5.1 (Pin_1)
- net GNDA: no longer names the net of J11.10 (Pin_10)
- new net: J2.2 (Pin_2), J3.2 (Pin_2), J4.2 (Pin_2), J5.2 (Pin_2)
- new net: R22.1, R23.1, R24.2
- no-connect marks 18 -> 21
Other:
- moved on the sheet: J10, J11

Commit message: More Consistent Naming
Parts:
- SW5: value Buck Control -> SW_DPDT_x2
Changed lines of the file:
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@@
       (effects (font (size 1.27 1.27)) (justify right))
     )
-    (property "Value" "Buck Control" (at 312.42 196.85 90)
+    (property "Value" "SW_DPDT_x2" (at 312.42 196.85 90)
       (effects (font (size 1.27 1.27)) (justify right))
     )
